Commit message: 1.mujoco仿真添加SimulationReset服务 2.添加rl使用示例，详见bxi_example_py 3.修改脚踝扭矩计算逻辑 4.增加urdf和xml的机器人质量准确性

File: bxi_hw_release/share/description/model/urdf/bot_elf/urdf/bot_elf.urdf (robot description, URDF)
Before this commit: robot bot_elf, 32 links, 31 joints
Links:
- link base_link: mass 8.1797 -> 8.50938212
- link l_ankle_x_link: mass 0.242076229237956 -> 0.36482443
- link l_ankle_y_link: mass 0.0230716180694964 -> 0.02307162
- link l_elb_y_link: mass 0.164832849485564 -> 0.16483285
- link l_hip_x_link: mass 1.52690683733997 -> 1.74956721
- link l_hip_y_link: mass 2.50086507860377 -> 2.500865
- link l_hip_z_link: mass 1.23681233828303 -> 1.23681234
- link l_knee_y_link: mass 1.42611317447382 -> 1.58922365
- link l_shld_x_link: mass 0.621968051279973 -> 0.62196805
- link l_shld_y_link: mass 0.397430898254414 -> 0.3974309
- link l_shld_z_link: mass 0.449112448185888 -> 0.44911245
- link r_ankle_x_link: mass 0.24207626222516 -> 0.36482447
- link r_ankle_y_link: mass 0.0230716180694967 -> 0.02307162
- link r_elb_y_link: mass 0.164832849485564 -> 0.16483285
- link r_hip_x_link: mass 1.52690683726889 -> 1.74956721
- link r_hip_y_link: mass 2.50086518492187 -> 2.50086544
- link r_hip_z_link: mass 1.23681232467206 -> 1.23681233
- link r_knee_y_link: mass 1.42506790131187 -> 1.5881784
- link r_shld_x_link: mass 0.621968051279973 -> 0.62196805
- link r_shld_y_link: mass 0.397430898254414 -> 0.39742959
- link r_shld_z_link: mass 0.449113232804568 -> 0.44911323
Joints:
- joint l_ankle_x_joint: limit lower=-0.349 upper=0.349 effort=5 velocity=20 -> lower=-0.349 upper=0.349 effort=7 velocity=20
- joint l_ankle_y_joint: limit lower=-1.134 upper=0.872 effort=10 velocity=20 -> lower=-1.134 upper=0.872 effort=14 velocity=20
- joint l_elb_y_joint: limit lower=-2 upper=2 effort=27 velocity=20 -> lower=-2 upper=0 effort=27 velocity=20
- joint l_hip_y_joint: limit lower=-2 upper=0.5 effort=38 velocity=20 -> lower=-2 upper=0.5 effort=50 velocity=20
- joint l_shld_x_joint: limit lower=-2 upper=2 effort=27 velocity=20 -> lower=-0.52 upper=2 effort=27 velocity=20
- joint l_shld_y_joint: limit lower=-2 upper=2 effort=27 velocity=20 -> lower=-1.5 upper=1.5 effort=27 velocity=20
- joint l_shld_z_joint: limit lower=-2 upper=2 effort=7 velocity=20 -> lower=-1.5 upper=1.5 effort=7 velocity=20
- joint r_ankle_x_joint: limit lower=-0.349 upper=0.349 effort=5 velocity=20 -> lower=-0.349 upper=0.349 effort=7 velocity=20
- joint r_ankle_y_joint: limit lower=-1.134 upper=0.872 effort=10 velocity=20 -> lower=-1.134 upper=0.872 effort=14 velocity=20
- joint r_elb_y_joint: limit lower=-2 upper=2 effort=27 velocity=20 -> lower=-2 upper=0 effort=27 velocity=20
- joint r_hip_y_joint: limit lower=-2 upper=0.5 effort=38 velocity=20 -> lower=-2 upper=0.5 effort=50 velocity=20
- joint r_shld_x_joint: limit lower=-2 upper=2 effort=27 velocity=20 -> lower=-2 upper=0.52 effort=27 velocity=20
- joint r_shld_y_joint: limit lower=-2 upper=2 effort=27 velocity=20 -> lower=-1.5 upper=1.5 effort=27 velocity=20
- joint r_shld_z_joint: limit lower=-2 upper=2 effort=7 velocity=20 -> lower=-1.5 upper=1.5 effort=7 velocity=20
